File: hardwaredesign/dxdash/bus.kicad_sch (KiCad schematic)
At the start: 9 parts, among them J3 CAN, Q4 BC556, Q6 BC546, U1 SN65HVD234

Commit message: controller board added features
Parts:
- renumbered J3 to J12, JP2 to JP4, JP3 to JP5, R1 to R2, R3 to R4, R5 to R6, U1 to U2
Changed lines of the file:
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@@
 		(dnp no)
 		(fields_autoplaced yes)
-		(property "Reference" "J3"
+		(property "Reference" "J12"
 			(at 116.84 59.055 0)
 			(effects
@@
 		(instances
 			(project "dxdash"
-				(path "/e63e39d7-6ac0-4ffd-8aa3-1841a4541b55/97d456cc-2984-45c2-9f4f-55359f773ff4"
-					(reference "J3")
-					(unit 1)
-				)
 				(path "/e63e39d7-6ac0-4ffd-8aa3-1841a4541b55/d59a343a-b7c9-47a9-9cba-f2e4ce551af7"
 					(reference "J12")
@@
 		(on_board yes)
 		(dnp no)
-		(property "Reference" "#PWR02"
+		(property "Reference" "#PWR05"
 			(at 102.87 59.69 0)
 			(effects
@@
 		(instances
 			(project "dxdash"
-				(path "/e63e39d7-6ac0-4ffd-8aa3-1841a4541b55/97d456cc-2984-45c2-9f4f-55359f773ff4"
-					(reference "#PWR02")
-					(unit 1)
-				)
 				(path "/e63e39d7-6ac0-4ffd-8aa3-1841a4541b55/d59a343a-b7c9-47a9-9cba-f2e4ce551af7"
 					(reference "#PWR05")
@@
 		)
 		(instances
-			(project ""
-				(path "/e63e39d7-6ac0-4ffd-8aa3-1841a4541b55/97d456cc-2984-45c2-9f4f-55359f773ff4"
-					(reference "Q5")
-					(unit 1)
-				)
+			(project "dxdash"
 				(path "/e63e39d7-6ac0-4ffd-8aa3-1841a4541b55/d59a343a-b7c9-47a9-9cba-f2e4ce551af7"
 					(reference "Q6")
@@
 		(on_board yes)
 		(dnp no)
-		(property "Reference" "R5"
+		(property "Reference" "R6"
 			(at 156.972 72.136 90)
 			(effects
@@
 		(instances
 			(project "dxdash"
-				(path "/e63e39d7-6ac0-4ffd-8aa3-1841a4541b55/97d456cc-2984-45c2-9f4f-55359f773ff4"
-					(reference "R5")
-					(unit 1)
-				)
 				(path "/e63e39d7-6ac0-4ffd-8aa3-1841a4541b55/d59a343a-b7c9-47a9-9cba-f2e4ce551af7"
 					(reference "R6")
@@
 		(dnp no)
 		(fields_autoplaced yes)
-		(property "Reference" "JP3"
+		(property "Reference" "JP5"
 			(at 44.45 67.3099 90)
 			(effects
@@
 		(instances
 			(project "dxdash"
-				(path "/e63e39d7-6ac0-4ffd-8aa3-1841a4541b55/97d456cc-2984-45c2-9f4f-55359f773ff4"
-					(reference "JP3")
-					(unit 1)
-				)
 				(path "/e63e39d7-6ac0-4ffd-8aa3-1841a4541b55/d59a343a-b7c9-47a9-9cba-f2e4ce551af7"
 					(reference "JP5")
@@
 		(dnp no)
 		(fields_autoplaced yes)
-		(property "Reference" "U1"
+		(property "Reference" "U2"
 			(at 69.2659 49.53 0)
 			(effects
@@
 		(instances
 			(project "dxdash"
-				(path "/e63e39d7-6ac0-4ffd-8aa3-1841a4541b55/97d456cc-2984-45c2-9f4f-55359f773ff4"
-					(reference "U1")
-					(unit 1)
-				)
 				(path "/e63e39d7-6ac0-4ffd-8aa3-1841a4541b55/d59a343a-b7c9-47a9-9cba-f2e4ce551af7"
 					(reference "U2")
@@
 		)
 		(instances
-			(project ""
-				(path "/e63e39d7-6ac0-4ffd-8aa3-1841a4541b55/97d456cc-2984-45c2-9f4f-55359f773ff4"
-					(reference "Q1")
-					(unit 1)
-				)
+			(project "dxdash"
 				(path "/e63e39d7-6ac0-4ffd-8aa3-1841a4541b55/d59a343a-b7c9-47a9-9cba-f2e4ce551af7"
 					(reference "Q4")
@@
 		(dnp no)
 		(fields_autoplaced yes)
-		(property "Reference" "JP2"
+		(property "Reference" "JP4"
 			(at 83.82 55.8799 90)
 			(effects
@@
 		(instances
 			(project "dxdash"
-				(path "/e63e39d7-6ac0-4ffd-8aa3-1841a4541b55/97d456cc-2984-45c2-9f4f-55359f773ff4"
-					(reference "JP2")
-					(unit 1)
-				)
 				(path "/e63e39d7-6ac0-4ffd-8aa3-1841a4541b55/d59a343a-b7c9-47a9-9cba-f2e4ce551af7"
 					(reference "JP4")
@@
 		(on_board yes)
 		(dnp no)
-		(property "Reference" "#PWR03"
+		(property "Reference" "#PWR06"
 			(at 67.31 74.93 0)
 			(effects
@@
 		(instances
 			(project "dxdash"
-				(path "/e63e39d7-6ac0-4ffd-8aa3-1841a4541b55/97d456cc-2984-45c2-9f4f-55359f773ff4"
-					(reference "#PWR03")
-					(unit 1)
-				)
 				(path "/e63e39d7-6ac0-4ffd-8aa3-1841a4541b55/d59a343a-b7c9-47a9-9cba-f2e4ce551af7"
 					(reference "#PWR06")
@@
 		(on_board yes)
 		(dnp no)
-		(property "Reference" "#PWR04"
+		(property "Reference" "#PWR07"
 			(at 46.99 80.01 0)
 			(effects
@@
 		(instances
 			(project "dxdash"
-				(path "/e63e39d7-6ac0-4ffd-8aa3-1841a4541b55/97d456cc-2984-45c2-9f4f-55359f773ff4"
-					(reference "#PWR04")
-					(unit 1)
-				)
 				(path "/e63e39d7-6ac0-4ffd-8aa3-1841a4541b55/d59a343a-b7c9-47a9-9cba-f2e4ce551af7"
 					(reference "#PWR07")
@@
 		(on_board yes)
 		(dnp no)
-		(property "Reference" "#PWR08"
+		(property "Reference" "#PWR09"
 			(at 170.18 82.55 0)
 			(effects
@@
 		(instances
 			(project "dxdash"
-				(path "/e63e39d7-6ac0-4ffd-8aa3-1841a4541b55/97d456cc-2984-45c2-9f4f-55359f773ff4"
-					(reference "#PWR08")
-					(unit 1)
-				)
 				(path "/e63e39d7-6ac0-4ffd-8aa3-1841a4541b55/d59a343a-b7c9-47a9-9cba-f2e4ce551af7"
 					(reference "#PWR09")
@@
 		(on_board yes)
 		(dnp no)
-		(property "Reference" "R1"
+		(property "Reference" "R2"
 			(at 81.28 69.85 0)
 			(effects
@@
 		(instances
 			(project "dxdash"
-				(path "/e63e39d7-6ac0-4ffd-8aa3-1841a4541b55/97d456cc-2984-45c2-9f4f-55359f773ff4"
-					(reference "R1")
-					(unit 1)
-				)
 				(path "/e63e39d7-6ac0-4ffd-8aa3-1841a4541b55/d59a343a-b7c9-47a9-9cba-f2e4ce551af7"
 					(reference "R2")
@@
 		(on_board yes)
 		(dnp no)
-		(property "Reference" "R3"
+		(property "Reference" "R4"
 			(at 173.228 52.324 0)
 			(effects
@@
 		(instances
 			(project "dxdash"
-				(path "/e63e39d7-6ac0-4ffd-8aa3-1841a4541b55/97d456cc-2984-45c2-9f4f-55359f773ff4"
-					(reference "R3")
-					(unit 1)
-				)
 				(path "/e63e39d7-6ac0-4ffd-8aa3-1841a4541b55/d59a343a-b7c9-47a9-9cba-f2e4ce551af7"
 					(reference "R4")

Commit message: added switch inputs. Layout preparation.
Parts:
- JP4: footprint (none) -> Jumper:SolderJumper-2_P1.3mm_Open_TrianglePad1.0x1.5mm
- JP5: footprint (none) -> Jumper:SolderJumper-3_P1.3mm_Open_Pad1.0x1.5mm_NumberLabels
Changed lines of the file:
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@@
 			)
 		)
-		(property "Footprint" ""
+		(property "Footprint" "Jumper:SolderJumper-3_P1.3mm_Open_Pad1.0x1.5mm_NumberLabels"
 			(at 46.99 68.58 0)
 			(effects
@@
 			)
 		)
-		(property "Footprint" ""
+		(property "Footprint" "Jumper:SolderJumper-2_P1.3mm_Open_TrianglePad1.0x1.5mm"
 			(at 81.28 57.15 0)
 			(effects

Commit message: more layout
Parts:
- removed J12: CAN, Connector_PinHeader_2.54mm:PinHeader_1x03_P2.54mm_Vertical, symbol Connector:Conn_01x03_Pin
Changed lines of the file:
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@@
 	(paper "A4")
-	(junction
-		(at 86.36 68.58)
-		(diameter 0)
-		(color 0 0 0 0)
-	)
 	(junction
 		(at 81.28 53.34)
@@
 	)
 	(junction
-		(at 86.36 53.34)
-		(diameter 0)
-		(color 0 0 0 0)
-	)
-	(junction
 		(at 67.31 68.58)
 		(diameter 0)
@@
 	(wire
 		(pts
-			(xy 81.28 68.58) (xy 86.36 68.58)
-		)
-		(stroke
-			(width 0)
-			(type default)
-		)
-	)
-	(wire
-		(pts
-			(xy 81.28 53.34) (xy 86.36 53.34)
+			(xy 81.28 68.58) (xy 90.17 68.58)
+		)
+		(stroke
+			(width 0)
+			(type default)
+		)
+	)
+	(wire
+		(pts
+			(xy 81.28 53.34) (xy 90.17 53.34)
 		)
 		(stroke
@@
 	(wire
 		(pts
-			(xy 90.17 72.39) (xy 86.36 72.39)
-		)
-		(stroke
-			(width 0)
-			(type default)
-		)
-	)
-	(wire
-		(pts
 			(xy 77.47 58.42) (xy 77.47 53.34)
 		)
@@
 	(wire
 		(pts
-			(xy 110.49 53.34) (xy 110.49 57.15)
-		)
-		(stroke
-			(width 0)
-			(type default)
-		)
-	)
-	(wire
-		(pts
 			(xy 53.34 55.88) (xy 57.15 55.88)
 		)
@@
 	(wire
 		(pts
-			(xy 86.36 72.39) (xy 86.36 68.58)
-		)
-		(stroke
-			(width 0)
-			(type default)
-		)
-	)
-	(wire
-		(pts
 			(xy 57.15 68.58) (xy 67.31 68.58)
 		)
@@
 	(wire
 		(pts
-			(xy 86.36 53.34) (xy 110.49 53.34)
-		)
-		(stroke
-			(width 0)
-			(type default)
-		)
-	)
-	(wire
-		(pts
 			(xy 81.28 67.31) (xy 81.28 68.58)
 		)
@@
 	(wire
 		(pts
-			(xy 110.49 68.58) (xy 110.49 62.23)
-		)
-		(stroke
-			(width 0)
-			(type default)
-		)
-	)
-	(wire
-		(pts
 			(xy 170.18 55.88) (xy 170.18 63.5)
 		)
@@
 	(wire
 		(pts
-			(xy 91.44 48.26) (xy 86.36 48.26)
-		)
-		(stroke
-			(width 0)
-			(type default)
-		)
-	)
-	(wire
-		(pts
-			(xy 86.36 68.58) (xy 110.49 68.58)
-		)
-		(stroke
-			(width 0)
-			(type default)
-		)
-	)
-	(wire
-		(pts
 			(xy 173.99 46.99) (xy 170.18 46.99)
 		)
@@
 	(wire
 		(pts
-			(xy 86.36 48.26) (xy 86.36 53.34)
-		)
-		(stroke
-			(width 0)
-			(type default)
-		)
-	)
-	(wire
-		(pts
 			(xy 170.18 73.66) (xy 170.18 76.2)
 		)
@@
 		(pts
 			(xy 50.8 68.58) (xy 50.8 60.96)
-		)
-		(stroke
-			(width 0)
-			(type default)
-		)
-	)
-	(wire
-		(pts
-			(xy 110.49 59.69) (xy 109.22 59.69)
 		)
 		(stroke
@@
 	(global_label "CANH"
 		(shape input)
-		(at 91.44 48.26 0)
+		(at 90.17 53.34 0)
 		(fields_autoplaced yes)
 		(effects
@@
 		)
 		(property "Intersheetrefs" "${INTERSHEET_REFS}"
-			(at 99.3654 48.26 0)
+			(at 98.0954 53.34 0)
 			(effects
 				(font
@@
 	(global_label "CANL"
 		(shape input)
-		(at 90.17 72.39 0)
+		(at 90.17 68.58 0)
 		(fields_autoplaced yes)
 		(effects
@@
 		)
 		(property "Intersheetrefs" "${INTERSHEET_REFS}"
-			(at 97.793 72.39 0)
+			(at 97.793 68.58 0)
 			(effects
 				(font
@@
 			)
 		)
-	)
-	(symbol
-		(lib_id "Connector:Conn_01x03_Pin")
-		(at 115.57 59.69 180)
-		(unit 1)
-		(exclude_from_sim no)
-		(in_bom yes)
-		(on_board yes)
-		(dnp no)
-		(fields_autoplaced yes)
-		(property "Reference" "J12"
-			(at 116.84 59.055 0)
-			(effects
-				(font
-					(size 1.27 1.27)
-				)
-				(justify right)
-			)
-		)
-		(property "Value" "CAN"
-			(at 116.84 61.595 0)
-			(effects
-				(font
-					(size 1.27 1.27)
-				)
-				(justify right)
-			)
-		)
-		(property "Footprint" "Connector_PinHeader_2.54mm:PinHeader_1x03_P2.54mm_Vertical"
-			(at 115.57 59.69 0)
-			(effects
-				(font
-					(size 1.27 1.27)
-				)
-				(hide yes)
-			)
-		)
-		(property "Datasheet" "~"
-			(at 115.57 59.69 0)
-			(effects
-				(font
-					(size 1.27 1.27)
-				)
-				(hide yes)
-			)
-		)
-		(property "Description" ""
-			(at 115.57 59.69 0)
-			(effects
-				(font
-					(size 1.27 1.27)
-				)
-				(hide yes)
-			)
-		)
-		(pin "1"
-		)
-		(pin "2"
-		)
-		(pin "3"
-		)
-		(instances
-			(project "dxdash"
-				(path "/e63e39d7-6ac0-4ffd-8aa3-1841a4541b55/d59a343a-b7c9-47a9-9cba-f2e4ce551af7"
-					(reference "J12")
-					(unit 1)
-				)
-			)
-		)
-	)
-	(symbol
-		(lib_id "power:GND")
-		(at 109.22 59.69 270)
-		(unit 1)
-		(exclude_from_sim no)
-		(in_bom yes)
-		(on_board yes)
-		(dnp no)
-		(property "Reference" "#PWR05"
-			(at 102.87 59.69 0)
-			(effects
-				(font
-					(size 1.27 1.27)
-				)
-				(hide yes)
-			)
-		)
-		(property "Value" "GND"
-			(at 106.68 59.69 90)
-			(effects
-				(font
-					(size 1.27 1.27)
-				)
-				(justify right)
-			)
-		)
-		(property "Footprint" ""
-			(at 109.22 59.69 0)
-			(effects
-				(font
-					(size 1.27 1.27)
-				)
-				(hide yes)
-			)
-		)
-		(property "Datasheet" ""
-			(at 109.22 59.69 0)
-			(effects
-				(font
-					(size 1.27 1.27)
-				)
-				(hide yes)
-			)
-		)
-		(property "Description" ""
-			(at 109.22 59.69 0)
-			(effects
-				(font
-					(size 1.27 1.27)
-				)
-				(hide yes)
-			)
-		)
-		(pin "1"
-		)
-		(instances
-			(project "dxdash"
-				(path "/e63e39d7-6ac0-4ffd-8aa3-1841a4541b55/d59a343a-b7c9-47a9-9cba-f2e4ce551af7"
-					(reference "#PWR05")
-					(unit 1)
-				)
-			)
-		)
